Commit message: minor changes and license specification

File: robucar_description/urdf/robucar.urdf.xacro (robot description, xacro)
@@ -24,5 +24,5 @@
     <xacro:property name="carLength" value="2.0" />
     <xacro:property name="carWidth" value="1.00" />
-    <xacro:property name="carHeight" value="0.6" />
+    <xacro:property name="carHeight" value="0.5" />
     <xacro:property name="wheelRadius" value="0.2125" />
     <xacro:property name="wheelWidth" value="0.125" />
@@ -31,9 +31,15 @@
     	<color rgba="1.0 0 0 1.0"/>
     </material>
+    <material name="Yellow">
+        <color rgba="1.0 1.0 0 1.0"/>
+    </material>
+    <material name="Grey">
+        <color rgba="0.25 0.25 0.25 1.0"/>
+    </material>
     <material name="Green">
     	<color rgba="0 1.0 0 1.0"/>
     </material>
     <material name="Blue">
-    	<color rgba="0 0 1.0 0.5"/>
+    	<color rgba="0 0 1.0 1.0"/>
     </material>
     <material name="Black">
@@ -55,5 +61,5 @@
                 <box size="${carLength} ${carWidth} ${carHeight}" />
             </geometry>
-            <material name="Red"/>
+            <material name="Grey"/>
         </visual>
         <collision>
@@ -65,5 +71,5 @@
     </link>
     <gazebo reference="base_link">
-        <material>Gazebo/Red</material>
+        <material>Gazebo/Grey</material>
     </gazebo>
     <!-- Front link of Ackermann -->
@@ -93,5 +99,5 @@
     </link>
     <gazebo reference="front_link">
-        <material>Gazebo/Green</material>
+        <material>Gazebo/Black</material>
     </gazebo>
     <!-- a link aligned with the steer direction -->
@@ -114,5 +120,5 @@
                 <box size="${carLength*0.1} ${carWidth*0.133} ${carHeight*0.05}" />
             </geometry>
-            <material name="Green"/>
+            <material name="Black"/>
         </visual>
         <collision>
@@ -124,5 +130,5 @@
     </link>
     <gazebo reference="steer_link">
-        <material>Gazebo/Green</material>
+        <material>Gazebo/Black</material>
     </gazebo>
     <!-- the left Ackermann bar -->
@@ -145,5 +151,5 @@
                 <box size="${carLength*0.1} ${carWidth*0.133} ${carHeight*0.05}" />
             </geometry>
-            <material name="Green"/>
+            <material name="Black"/>
         </visual>
         <collision>
@@ -155,5 +161,5 @@
     </link>
     <gazebo reference="front_left_bar_link">
-        <material>Gazebo/Green</material>
+        <material>Gazebo/Black</material>
     </gazebo>
     <!-- the right Ackermann bar -->
@@ -176,5 +182,5 @@
                 <box size="${carLength*0.1} ${carWidth*0.133} ${carHeight*0.05}" />
             </geometry>
-            <material name="Green"/>
+            <material name="Black"/>
         </visual>
         <collision>
@@ -186,5 +192,5 @@
     </link>
     <gazebo reference="front_right_bar_link">
-        <material>Gazebo/Green</material>
+        <material>Gazebo/Black</material>
     </gazebo>
 	<!-- the front left wheel -->
@@ -206,5 +212,5 @@
                 <cylinder radius="${wheelRadius}" length="${wheelWidth}" />
             </geometry>
-            <material name="Green"/>
+            <material name="Black"/>
         </visual>
         <collision>
@@ -216,5 +222,5 @@
     </link>
     <gazebo reference="front_left_wheel_link">
-        <material>Gazebo/Green</material>
+        <material>Gazebo/Black</material>
     </gazebo>
 	<!-- the front right wheel -->
@@ -236,5 +242,5 @@
                 <cylinder radius="${wheelRadius}" length="${wheelWidth}" />
             </geometry>
-            <material name="Green"/>
+            <material name="Black"/>
         </visual>
         <collision>
@@ -246,5 +252,5 @@
     </link>
     <gazebo reference="front_right_wheel_link">
-        <material>Gazebo/Green</material>
+        <material>Gazebo/Black</material>
         <turnGravityOff>false</turnGravityOff>
     </gazebo>
@@ -267,5 +273,5 @@
                 <box size="${carLength*0.05} ${carWidth} ${carHeight*0.1}" />
             </geometry>
-            <material name="Green"/>
+            <material name="Black"/>
         </visual>
         <collision>
@@ -276,5 +282,5 @@
     </link>
     <gazebo reference="front_link">
-        <material>Gazebo/Green</material>
+        <material>Gazebo/Black</material>
     </gazebo>
     <gazebo reference="ackermann_bar_link">
@@ -401,11 +407,12 @@
             </inertial>
             <visual>
-                <origin rpy="0 0 0" xyz="0.679 0 0.4"/>
+                <origin rpy="0 0 0" xyz="1.0 0 0.4"/>
                 <geometry>
                     <box size="0.18 0.18 0.18"/>
                 </geometry>
+                <material name="Blue"/>
             </visual>
             <collision>
-                <origin rpy="0 0 0" xyz="0.679 0 0.025"/>
+                <origin rpy="0 0 0" xyz="1.0 0 0.4"/>
                 <geometry>
                     <box size="0.18 0.18 0.18"/>
@@ -429,4 +436,5 @@
                     <cylinder radius="0.0229" length="0.028"/>
                 </geometry>
+                <material name="Blue"/>
             </visual>
             <collision>
@@ -444,6 +452,6 @@
                 <origin>0.0 0.0 0.0</origin>
                 <displayRays>false</displayRays>
-                <minAngle>-135</minAngle>
-                <maxAngle> 135</maxAngle>
+                <minAngle>0</minAngle>
+                <maxAngle>180</maxAngle>
                 <minRange>0.06</minRange>
                 <maxRange>4.0</maxRange>
@@ -461,8 +469,8 @@
         </gazebo>
         <gazebo reference="laser_base_link">
-            <material>Gazebo/Black</material>
+            <material>Gazebo/Blue</material>
         </gazebo>
         <gazebo reference="laser">
-            <material>Gazebo/Black</material>
+            <material>Gazebo/Blue</material>
         </gazebo>
 </robot>
